File: pcb/MEMSpcb.kicad_sch (KiCad schematic)
At the start: 4 parts, among them J2 Conn_02x04_Odd_Even

Commit message: added bom and stuff
Parts:
- C1: LCSC (none) -> C122257
- MK1: LCSC (none) -> C20344623
- R1: LCSC (none) -> C270298
